Commit message: Create to different pkg urg_node and urg_description

File: urg_description/urdf/hokuyo_urg_04lx_ug01_laser.urdf.xacro (robot description, xacro)
@@ -8,5 +8,5 @@
 -->
 <robot xmlns:xacro="http://ros.org/wiki/xacro">
-  <xacro:include filename="$(find urg_node)/urdf/hokuyo_urg_04lx_ug01_laser.gazebo.xacro" />
+  <xacro:include filename="$(find urg_description)/urdf/hokuyo_urg_04lx_ug01_laser.gazebo.xacro" />
   <xacro:macro name="hokuyo_urg_04lx_ug01_laser" params="name parent *origin ros_topic update_rate min_angle max_angle">
     <link name="${name}_link" type="laser">
@@ -21,5 +21,5 @@
         <origin xyz="0 0 0" rpy="0 0 0" />
         <geometry>
-          <mesh filename="package://urg_node/meshes/hokuyo_urg_04lx_ug01.stl"/>
+          <mesh filename="package://urg_description/meshes/hokuyo_urg_04lx_ug01.stl"/>
         </geometry>
         <material name="DarkGrey">

File: urg_description/urdf/hokuyo_utm30lx.urdf.xacro (robot description, xacro)
@@ -17,5 +17,5 @@
           <origin xyz="0 0 0" rpy="0 0 0" />
           <geometry>
-          <mesh filename="package://urg_node/meshes/hokuyo_utm30lx/hokuyo_utm_30lx.dae"/>
+          <mesh filename="package://urg_description/meshes/hokuyo_utm30lx/hokuyo_utm_30lx.dae"/>
         </geometry>
         </visual>
@@ -24,5 +24,5 @@
           <geometry>
           <box size="0.058 0.058 0.087" />
-          <!--<mesh filename="package://urg_node/meshes/hokuyo_utm30lx/hokuyo_utm_30lx.stl"/>-->
+          <!--<mesh filename="package://urg_description/meshes/hokuyo_utm30lx/hokuyo_utm_30lx.stl"/>-->
         </geometry>
         </collision>
